Commit message: Re-factored and fixed visual tools demo!

File: resources/rrbot.urdf (robot description, URDF)
Before this commit: robot rrbot, 4 links, 3 joints
Links:
- removed link world
- added link base_link
Joints:
- joint fixed: origin (none) -> xyz=0 0 0 rpy=0 0 0; parent world -> base_link
